File: pcb/Drone/Drone.kicad_sch (KiCad schematic)
At the start: 31 parts, among them J1 USB_C_Receptacle_USB2.0_16P, J2 Conn_01x22_Pin, J3 Conn_01x22_Pin, Q1 NPN, Q2 NPN, U2 CH343P, U3 AMS1117-3.3

Commit message: update pcb
Parts:
- removed D6: D_Small, symbol Device:D_Small
- removed R2, R4: R_Small_US, symbol Device:R_Small_US
- added R10: 10K, symbol Device:R_Small_US
- added U4: USBLC6-2SC6, Package_TO_SOT_SMD:SOT-23-6, symbol Power_Protection:USBLC6-2SC6
- added U5: CH343P, Package_DFN_QFN:WCH_QFN-16-1EP_3x3mm_P0.5mm_EP1.8x1.8mm, symbol Interface_USB:CH343P
- C10, C9: value C_Small -> C
- C5: value C_Small -> 0.1u
- C6: value C_Small -> 1u
- C7: value C_Small -> 10u
- R3, R5, R6, R7: value R_Small_US -> 10K
- R8: value R_Small_US -> R
Connections:
- net VDD33 is gone; now on net +3V3: C10.1, C4.1, C5.1, C6.1, J2.1 (Pin_1), J2.2 (Pin_2), R8.1, U2.1 (VIO), U3.2 (VO)
- net D+: now also U4.4 (I/O2), U5.7 (UD+); no longer J1.A7 (D-), J1.B7 (D-)
- net D-: now also U4.6 (I/O1), U5.8 (UD-); no longer J1.A6 (D+), J1.B6 (D+)
- net DTR: now also U5.12 (~{DTR})
- net GND: now also J1.SH (SHIELD), U1.40 (GND), R10.2, U4.2 (GND), U5.17 (GND_EPAD), U5.2 (GND)
- net RTS: now also U5.13 (~{RTS})
- net U0RXD: now also U5.4 (TXD)
- net U0TXD: now also U5.5 (RXD)
- net VBUSB: no longer J1.A4 (VBUS), J1.A9 (VBUS), J1.B4 (VBUS), J1.B9 (VBUS), U2.9 (VBUS)
- net +3V3: now reaches R3.1, U1.2 (3V3)
- net at J1.B5 (CC2): now also R10.1
- net 5V renamed +5V
- new net: J1.A7 (D-), J1.B7 (D-), U4.1 (I/O1)
- new net: J1.A6 (D+), J1.B6 (D+), U4.3 (I/O2)
- new net VBUS: J1.A4 (VBUS), J1.A9 (VBUS), J1.B4 (VBUS), J1.B9 (VBUS), U2.9 (VBUS), U4.5 (VBUS), U5.9 (VBUS)
- no-connect marks 0 -> 2
Other:
- moved on the sheet: BOOT1, C1, C10, C2, C5, C6, C7, C9, D3, D5, J2, J3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

Commit message: schematic: battery and power selection
Parts:
- removed C3, C4, C8: C_Small, symbol Device:C_Small
- removed D3: LED, symbol Device:LED
- removed D5: D_Small, symbol Device:D_Small
- removed J2, J3: Conn_01x22_Pin, symbol Connector:Conn_01x22_Pin
- removed R9: R_Small_US, symbol Device:R_Small_US
- removed U2, U5: CH343P, Package_DFN_QFN:WCH_QFN-16-1EP_3x3mm_P0.5mm_EP1.8x1.8mm, symbol Interface_USB:CH343P
- removed U3: AMS1117-3.3, Package_TO_SOT_SMD:SOT-223-3_TabPin2, symbol Regulator_Linear:AMS1117-3.3
- added C11: 1u, symbol Device:C_Small
- added C12, C13: 0.1u, symbol Device:C_Small
- added D1: Red, symbol Device:LED_Small
- added D3: BAT54C, Package_TO_SOT_SMD:SOT-23, symbol Diode:BAT54C
- added D4, D5: D, symbol Device:D_Schottky
- added H1, H2, H3, H4: MountingHole, symbol Mechanical:MountingHole
- added J2, J3, J4, J6: XH2.54, symbol Connector:Conn_01x03_Pin
- added J5: Socket, symbol Connector:Conn_01x02_Socket
- added Q3: Si2301, symbol Simulation_SPICE:PMOS
- added R1: 4K7, symbol Device:R_Small_US
- added R11: 47K5, symbol Device:R_Small_US
- added R12: 100, symbol Device:R_Small_US
- added R13: 1K, symbol Device:R_Small_US
- added R14, R2: 10K, symbol Device:R_Small_US
- added R4: 22K1, symbol Device:R_Small_US
- added U2: DW01A, Package_TO_SOT_SMD:SOT-23-6, symbol Battery_Management:DW01A
- added U5: (no value), Package_TO_SOT_SMD:TSOT-23-6, symbol Battery_Management_ICs:8205
- added U6: (no value), Package_DFN_QFN:QFN-28-1EP_5x5mm_P0.5mm_EP3.1x3.1mm, symbol USB_to_UART:CP2102_QFN28_5x5mm
- added U8: ME6211C33M5, Package_TO_SOT_SMD:SOT-23-5, symbol Regulator_Linear:ME6211C33M5
- C10, C9: value C -> 22u
- J1: footprint (none) -> Connector_USB:USB_C_Receptacle_GCT_USB4105-xx-A_16P_TopMnt_Horizontal
- Q1, Q2: value NPN -> SS0805
- R10, R5: value 10K -> 5K1
- R8: value R -> 2K
Connections:
- net +5V is gone; now on an unnamed net: C9.1
- net +3V3: now also C11.1, R1.2, U6.6 (VDD), U6.7 (REGIN), U8.5 (V_{OUT}); no longer R8.1
- net DTR: now also U6.28 (DTR)
- net GND: now also C11.2, C12.2, D1.1 (K), J2.1 (Pin_1), J3.1 (Pin_1), J4.1 (Pin_1), J6.1 (Pin_1), R11.2, R13.2, R14.1, R2.2, U5.3 (S2), U6.3 (GND), U8.2 (V_{SS})
- net RTS: now also U6.24 (RTS)
- net VBUS: now also D3.2, D4.2 (A), R4.1
- net at R8.2: now also D4.1 (K), D5.1 (K), Q3.3 (S), U8.1 (V_{IN})
- net at J1.A5 (CC1): now also R10.1; no longer R5.1
- net at J1.B5 (CC2): now also R5.1; no longer R10.1
- net D+ renamed USB_D+
- net USB_D+: now also U6.4 (D+)
- net D- renamed USB_D-
- net USB_D-: now also U6.5 (D-)
- new net: C13.2, J5.2 (Pin_2), U2.6 (GND)
- new net: C12.1, R11.1, R4.2, U6.8 (VBUS)
- new net: C13.1, R12.2, U2.5 (VCC)
- new net: D3.3, Q3.2 (G), R14.2
- new net: R13.1, U2.2 (CS)
- new net: R2.1, U6.11 (~{SUSPEND})
- new net: R1.1, U6.9 (~{RST})
- new net: D1.2 (A), R8.1
- new net: U2.1 (OD), U5.6 (G1)
- new net: U2.3 (OC), U5.4 (G2)
- new net +BATT: J5.1 (Pin_1), Q3.1 (D), R12.1
- new net PWM1: J2.3 (Pin_3)
- new net PWM2: J3.3 (Pin_3)
- new net PWM3: J4.3 (Pin_3)
- new net PWM4: J6.3 (Pin_3)
- new net RXD: U6.25 (RXD)
- new net TXD: U6.26 (TXD)
- new net VBEC: D3.1, D5.2 (A), J2.2 (Pin_2)
- no-connect marks 2 -> 16
Other:
- note added: "BATTERY PROTECTION"
- note added: "ESCs"
- note added: "Lipo 1S 3.7-4.2V"
- note added: "MCU"
- note added: "MOUNTING HOLES"
- note added: "POWER SELECTION & REGULATING"
- note added: "USB & BOOT"
- note removed: "BOOT"
- note removed: "ESP32"
- note removed: "POWER"
- company: (none) -> Metrology Lab HCMUT
- title: (none) -> OISP Drone: Flight Controller
- moved on the sheet: BOOT1, C1, C10, C2, C5, C6, C7, J1, Q1, Q2, R3, R6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

Commit message: added footprints
Parts:
- removed BOOT1, RST1: SW_Push, symbol Switch:SW_Push
- added C14: 0.1u, Capacitor_SMD:C_0402_1005Metric, symbol Device:C_Small
- added D2: WS2812B-2020, LED_SMD:LED_WS2812B-2020_PLCC4_2.0x2.0mm, symbol LED:WS2812B-2020
- added J10, J7, J9: JST1.25, JST_1.25mm_RA_SMD:JST_1.25mm_RA_SMD_4P, symbol Connector:Conn_01x04_Socket
- added J8: JST1.25, JST_1.25mm_RA_SMD:JST_1.25mm_RA_SMD_8P, symbol Connector:Conn_01x07_Socket
- added SW1: RST, Button_Switch_SMD:SW_SPST_EVQP2_MiddlePushTravel_H2.5mm, symbol Switch:SW_Push
- added SW2: BOOT, Button_Switch_SMD:SW_SPST_EVQP2_MiddlePushTravel_H2.5mm, symbol Switch:SW_Push
- C1, C10, C11, C12, C13, C2, C5, C6, C7, C9: footprint (none) -> Capacitor_SMD:C_0402_1005Metric
- D1: footprint (none) -> LED_SMD:LED_0805_2012Metric
- D3: Supplier (none) -> https://chipn24.com/25-con-diode-schottky-dan-bat54c-kl3-so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
- H1, H2, H3, H4: value MountingHole -> M3; footprint (none) -> MountingHole:MountingHole_3.2mm_M3_Pad
- J1: Supplier (none) -> https://chipn24.com/dau-usb-type-c-v1-16p-usb-3-1-truyen-ta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
- J2, J3, J4, J6: value XH2.54 -> JST1.25; footprint (none) -> JST_1.25mm_RA_SMD:JST_1.25mm_RA_SMD_3P
- J5: value Socket -> JST1.25; footprint (none) -> JST_1.25mm_RA_SMD:JST_1.25mm_RA_SMD_2P
- Q1, Q2: value SS0805 -> SS8050; footprint (none) -> Package_TO_SOT_SMD:SOT-23; Supplier (none) -> https://www.thegioiic.com/ss8050-y1-transistor-npn-25v-1-5a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
- Q3: footprint (none) -> Package_TO_SOT_SMD:SOT-23; Supplier (none) -> https://www.thegioiic.com/si2301ds-mosfet-kenh-p-20v-2-3a-s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
- R1, R10, R11, R12, R13, R14, R2, R3, R4, R5, R6, R7, R8: footprint (none) -> Resistor_SMD:R_0402_1005Metric
- U1: value (none) -> esp32s3_wroom1; Supplier (none) -> https://hshop.vn/mach-thu-phat-wifi-ble-soc-esp32-s3-esp32-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
- U2: Supplier (none) -> https://www.thegioiic.com/dw01a-ic-bao-ve-pin-1-cell-sot-23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
- U4: Supplier (none) -> https://icdayroi.com/usblc6-2sc6-tvs-diode-5-25v-17v-sot23-6
- U5: value (none) -> 8205; Supplier (none) -> https://chipn24.com/ic-dan-8205s-sot-23-6-smd-fs8205-8205-i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
- U6: value (none) -> CP2102
- U8: Supplier (none) -> https://chipn24.com/ic-dan-me6211-sot23-5-smd-me6211c33m5g-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
Connections:
- net +3V3: now also J10.1 (Pin_1), J7.1 (Pin_1), J8.1 (Pin_1), J9.1 (Pin_1)
- net +BATT: now also Q3.3 (D); no longer Q3.1 (D)
- net CHIP_PU: now also Q1.3 (C), SW1.2; no longer Q1.1 (C)
- net DTR: now also Q2.2 (E); no longer Q2.3 (E)
- net GND: now also C14.2, D2.2 (VSS), J10.2 (Pin_2), J7.2 (Pin_2), J8.2 (Pin_2), J9.2 (Pin_2), SW1.1, SW2.1
- net GPIO0: now also Q2.3 (C), SW2.2; no longer Q2.1 (C)
- net RTS: now also Q1.2 (E); no longer Q1.3 (E)
- net at R7.2: now also Q2.1 (B); no longer Q2.2 (B)
- net RGB_POW: now reaches C9.1, D4.1 (K), D5.1 (K), R8.2, U8.1 (V_{IN})
- net RGB_POW: now also Q3.2 (S), C14.1, D2.4 (VDD); no longer Q3.3 (S)
- net at R6.2: now also Q1.1 (B); no longer Q1.2 (B)
- net at D3.3, R14.2: now also Q3.1 (G); no longer Q3.2 (G)
- new net CS: J8.6 (Pin_6)
- new net GPIOx: J8.7 (Pin_7)
- new net MISO: J8.4 (Pin_4)
- new net MOSI: J8.3 (Pin_3)
- new net RGB: D2.3 (DIN)
- new net RX: J9.4 (Pin_4)
- new net SCK: J8.5 (Pin_5)
- new net SCL1: J10.3 (Pin_3), J7.3 (Pin_3)
- new net SDA1: J10.4 (Pin_4), J7.4 (Pin_4)
- new net TX: J9.3 (Pin_3)
- no-connect marks 16 -> 17
Other:
- note added: "CONNECTORS"
- note added: "I2C"
- note added: "SPI"
- note added: "UART"
- moved on the sheet: C11, C12, H1, J2, J3, J4, J6, Q1, Q2, R1, R11, R2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

Commit message: hi
Parts:
- added U3: GY-87, GY-87:GY-87, symbol GY-87:GY-87
Changed lines of the file:
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@@
+	)
+	(symbol
+		(lib_id "GY-87:GY-87")
+		(at 350.52 218.44 0)
+		(unit 1)
+		(body_style 1)
+		(exclude_from_sim no)
+		(in_bom yes)
+		(on_board yes)
+		(in_pos_files yes)
+		(dnp no)
+		(fields_autoplaced yes)
+		(property "Reference" "U3"
+			(at 349.885 190.5 0)
+			(show_name no)
+			(do_not_autoplace no)
+			(effects
+				(font
+					(size 1.27 1.27)
+				)
+			)
+		)
+		(property "Value" "GY-87"
+			(at 349.885 193.04 0)
+			(show_name no)
+			(do_not_autoplace no)
+			(effects
+				(font
+					(size 1.27 1.27)
+				)
+			)
+		)
+		(property "Footprint" "GY-87:GY-87"
+			(at 350.012 218.44 0)
+			(hide yes)
+			(show_name no)
+			(do_not_autoplace no)
+			(effects
+				(font
+					(size 1.27 1.27)
+				)
+			)
+		)
+		(property "Datasheet" ""
+			(at 350.52 218.44 0)
+			(hide yes)
+			(show_name no)
+			(do_not_autoplace no)
+			(effects
+				(font
+					(size 1.27 1.27)
+				)
+			)
+		)
+		(property "Description" ""
+			(at 350.52 218.44 0)
+			(hide yes)
+			(show_name no)
+			(do_not_autoplace no)
+			(effects
+				(font
+					(size 1.27 1.27)
+				)
+			)
+		)
+		(pin "3"
+		)
+		(pin "2"
+		)
+		(pin "1"
+		)
+		(pin "4"
+		)
+		(pin "5"
+		)
+		(pin "6"
+		)
+		(pin "8"
+		)
+		(pin "7"
+		)
+		(instances
+			(project "Drone"
+				(path "/5ef9835f-9784-4760-b509-6732c7d681d2"
+					(reference "U3")
+					(unit 1)
+				)
+			)
+		)
 	)
 	(symbol
