File: pcb/Drone/Drone.kicad_sch (KiCad schematic)
At the start: 63 parts, among them J1 USB_C_Receptacle_USB2.0_16P, J10 JST1.25, J2 JST1.25, J3 JST1.25, J4 JST1.25, J5 JST1.25, J6 JST1.25, J7 JST1.25, J8 JST1.25, J9 JST1.25, Q1 SS8050, Q2 SS8050, Q3 Si2301, SW1 RST, SW2 BOOT, U1 esp32s3_wroom1, U10 AP2112K-3.3, U2 DW01A, U4 USBLC6-2SC6, U5 8205, U6 CP2102, U9 ME6211C33M5

Commit message: footprint
Parts:
- added U3: Ra02, Drone:RA-01H, symbol RF:Ra02
- added U7: (no value), symbol custom_symbols:MicroSD
- added U8: GY-87, Drone:GY-87, symbol GY-87:GY-87
