File: pcb/Power_Monitor/Power_Monitor.kicad_sch (KiCad schematic)
At the start: 0 parts

Commit message: development: 3d, power board, fc
Parts:
- added C1, C2: 0.1u, Capacitor_SMD:C_0805_2012Metric, symbol Device:C
- added H1, H2: M3, MountingHole:MountingHole_3.2mm_M3_DIN965_Pad, symbol Mechanical:MountingHole
- added J1: XT60, Connector_AMASS:AMASS_XT60PW-M_1x02_P7.20mm_Horizontal, symbol Connector:Conn_01x02_Socket
- added J2: JST1.25, Local Footprints:JST_1.25mm_RA_SMD_4P, symbol Connector:Conn_01x04_Socket
- added J3, J4: Castellated Pad, symbol Connector:Conn_01x01_Socket
- added R2, R3: 1mR, Resistor_SMD:R_2512_6332Metric, symbol Device:R_US
- added R4, R5: 4.7R, Resistor_SMD:R_0402_1005Metric, symbol Device:R_US
- added R6, R7, R8: 10K, Resistor_SMD:R_0402_1005Metric, symbol Device:R_US
- added U1: INA226, Package_SO:TSSOP-10_3x3mm_P0.5mm, symbol Sensor_Energy:INA226
Connections:
- new net: J1.2 (Pin_2), R2.1, R3.1, R4.1, U1.8 (Vbus)
- new net: C1.1, R4.2, U1.10 (Vin+)
- new net: J4.1 (Pin_1), R2.2, R3.2, R5.1
- new net: R6.1, U1.3 (~{Alert})
- new net: C1.2, R5.2, U1.9 (Vin-)
- new net +3V3: C2.1, J2.1 (Pin_1), R6.2, R7.2, R8.2, U1.6 (VS)
- new net GND: C2.2, J1.1 (Pin_1), J2.2 (Pin_2), J3.1 (Pin_1), U1.7 (GND)
- new net SCL: J2.3 (Pin_3), R7.1, U1.5 (SCL)
- new net SDA: J2.4 (Pin_4), R8.1, U1.4 (SDA)
Other:
- note added: "+"
- note added: "-"
- note added: "Battery"
- note added: "Load"
- note added: "Mounting Holes"
- company: (none) -> Metrology Lab HCMUT
- title: (none) -> Modus Project: Power Monitor

Commit message: rtos architecture
Parts:
- added C3: 0.1u, Capacitor_SMD:C_0402_1005Metric, symbol Device:C
- added D2: SMAJ15A, Diode_SMD:D_SMA, symbol Diode:SMAJ15A
- added NT1: NetTie_2, NetTie:NetTie-2_SMD_Pad0.5mm, symbol Device:NetTie_2
- added R1: 10R, Resistor_SMD:R_0402_1005Metric, symbol Device:R_US
- C1, C2: footprint Capacitor_SMD:C_0805_2012Metric -> Capacitor_SMD:C_0402_1005Metric
- J3: footprint (none) -> Local Footprints:Castellated_pad_high_side
- J4: footprint (none) -> Local Footprints:Castellated_pad_low_side
Connections:
- net at J1.2 (Pin_2), R2.1, R3.1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: now also D2.1 (A1), R1.1; no longer U1.8 (Vbus)
- net at R2.2, R3.2, R5.1: now also J3.1 (Pin_1); no longer J4.1 (Pin_1)
- net GND renamed GND2
- net GND2: now also C3.2, NT1.2; no longer J1.1 (Pin_1), J3.1 (Pin_1)
- new net: C3.1, R1.2, U1.8 (Vbus)
- new net GND1: D2.2 (A2), J1.1 (Pin_1), J4.1 (Pin_1), NT1.1
Other:
- moved on the sheet: C2, H1, H2, J1, J2
