File: pcb/FC_v01/FC_v01.kicad_sch (KiCad schematic)
At the start: 85 parts, among them J1 USB_C_Receptacle_USB2.0_16P, J10 2.54mm, J11 2.54mm, J12 JST1.25, J13 JST1.25, J14 Micro_SD_Card_Det1, J15 2.54mm, J2 JST1.25, J3 JST1.25, J4 JST1.25, J5 JST1.25, J6 JST1.25, J8 JST1.25, J9 2.54mm, Q1 SS8050, Q2 SS8050, Q3 Si2301, SW1 BOOT, SW2 USER, SW3 RST, U1 USBLC6-2SC6, U2 CP2102, U3 GY-87, U4 DW01A, U5 8205, U6 AP2112K-3.3, U7 ME6211C33M5, U8 Ai-Thinker-Ra-02, U9 esp32s3_wroom1

Commit message: feat(mag-calib): implement full 3D rotated ellipsoid SIMD calibration and system-wide updates
- Implement 3D rotated and offset ellipsoid fitting (ellipsoid_fit.h/cpp) with Adam optimizer and analytical gradients
- Enforce full hardware SIMD acceleration via Matrix and Vec3 overloaded operators
- Normalize calibrated and filtered magnetometer output to unit sphere for EKF attitude estimation
- Add continuous tumble acquisition with spatial-thinning distance gating in task_calib_mag
- Forward user button clicks from FSM to signal calibration completion
- Add Option 11 to universal_flight_analyzer.py with RMSE convergence and 3D projection plots
- Consolidate firmware Layer 4 core directories (sensor, math, blackbox, telemetry, interface)
- Update Flash NVS storage driver and boot logging for 9-parameter magnetometer calibration
Other:
- title: Modus Project: Flight Controller -> OISP Project: Flight Controller
Changed lines of the file:
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@@
 	(paper "A3")
 	(title_block
-		(title "Modus Project: Flight Controller")
+		(title "OISP Project: Flight Controller")
 		(rev "v01")
 		(company "Metrology Lab HCMUT")
