File: pcb/FC_v02/FC_v02.kicad_pcb (KiCad board)
At the start: 4 copper layers, 50 x 50 mm, 87 parts, among them J1 USB_C_Receptacle_USB2.0_16P, J10 2.54mm, J11 2.54mm, J12 JST1.25, J13 JST1.25, J14 Micro_SD_Card_Det1, J2 JST1.25, J3 JST1.25, J4 JST1.25, J5 JST1.25, J6 JST1.25, J8 JST1.25, J9 2.54mm, Q1 SS8050, Q2 SS8050, Q3 Si2301, SW1 BOOT, SW2 USER, SW3 RST, U1 USBLC6-2SC6, U2 CP2102, U3 GY-87, U4 DW01A, U5 8205, U6 AP2112K-3.3, U7 ME6211C33M5, U8 Ai-Thinker-Ra-02, U9 esp32s3_wroom1

Commit message: feat(mag-calib): implement full 3D rotated ellipsoid SIMD calibration and system-wide updates
- Implement 3D rotated and offset ellipsoid fitting (ellipsoid_fit.h/cpp) with Adam optimizer and analytical gradients
- Enforce full hardware SIMD acceleration via Matrix and Vec3 overloaded operators
- Normalize calibrated and filtered magnetometer output to unit sphere for EKF attitude estimation
- Add continuous tumble acquisition with spatial-thinning distance gating in task_calib_mag
- Forward user button clicks from FSM to signal calibration completion
- Add Option 11 to universal_flight_analyzer.py with RMSE convergence and 3D projection plots
- Consolidate firmware Layer 4 core directories (sensor, math, blackbox, telemetry, interface)
- Update Flash NVS storage driver and boot logging for 9-parameter magnetometer calibration
Parts:
- J12, J6: value JST1.25 -> MX1.25; footprint Local Footprints:JST_1.25mm_RA_SMD_4P -> Local Footprints:MX_1.25mm_RA_SMD_4P
- J13: footprint Local Footprints:JST_1.25mm_RA_SMD_2P -> Local Footprints:MX_1.25mm_RA_SMD_2P
- J2, J3, J4, J5: value JST1.25 -> MX1.25; footprint Local Footprints:JST_1.25mm_RA_SMD_3P -> Local Footprints:MX_1.25mm_RA_SMD_3P
- J8: value JST1.25 -> MX1.25; footprint Local Footprints:JST_1.25mm_RA_SMD_8P -> Local Footprints:MX_1.25mm_RA_SMD_8P
- R22, R23: moved to F.Cu
- moved R22 29.4 mm to (153.5, 121.5)
- moved R23 26.9 mm to (156.5, 121.5), turned to 0 degrees
- moved J6 23.6 mm to (150.4, 123.2), turned to 0 degrees
- moved J4 23.4 mm to (172.8, 114.5), turned to 90 degrees
- moved J3 0.70 mm to (139.4, 123.2)
- moved J12 0.35 mm to (162.4, 123.2)
- moved U3 0.07 mm to (148.2, 100.7)
Connections:
- J2 pad 3: /ESC_PWM3 -> /ESC_PWM4
- J3 pad 2: unconnected-(J3-Pin_2-Pad2) -> VBEC
- J4 pad 2: VBEC -> unconnected-(J4-Pin_2-Pad2)
- J4 pad 3: /ESC_PWM1 -> /ESC_PWM3
- J5 pad 3: /ESC_PWM4 -> /ESC_PWM1
- J6 pad 3: /SCL1 -> /JTAG_D+
- J6 pad 4: /SDA1 -> /JTAG_D-
- R22 pad 1: /SCL1 -> /JTAG_D+
- R23 pad 1: /SDA1 -> /JTAG_D-
- U9 pad 13: /ESC_PWM2 -> /JTAG_D-
- U9 pad 14: /DRDY -> /JTAG_D+
- U9 pad 15: /ESC_PWM1 -> /ESC_PWM2
- U9 pad 33: /SDA1 -> /ESC_PWM3
- U9 pad 34: /SCL1 -> /RF_RST
- U9 pad 35: /RF_RST -> /DRDY
- U9 pad 39: /ESC_PWM3 -> /ESC_PWM4
- U9 pad 4: /ESC_PWM4 -> /ESC_PWM1
Routing:
- net /SCL1: track 42.2 -> 0.00 mm, vias 2 -> 0
- net /SDA1: track 39.9 -> 0.00 mm, vias 2 -> 0
- net /JTAG_D-: track 0.00 -> 33.9 mm, vias 0 -> 2
- net /JTAG_D+: track 0.00 -> 32.6 mm, vias 0 -> 2
- net /DRDY: track 23.6 -> 50.4 mm, vias 1 -> 2
- net /ESC_PWM1: track 27.5 -> 10.8 mm, vias 2 -> 0
- net /ESC_PWM4: track 10.8 -> 23.1 mm, vias 0 -> 2
- net VBEC: track 9.82 -> 21.3 mm
- net /ESC_PWM3: track 23.1 -> 30.8 mm
- net +3V3: track 139.2 -> 144.2 mm, vias 9 -> 8
- net /ESC_PWM2: track 37.3 -> 33.2 mm
- net GND: track 84.1 -> 87.1 mm, vias 44 -> 43
- net /RF_RST: track 36.5 -> 34.5 mm
- net +3V3_SENS: track 37.3 -> 38.6 mm
- net +5V: track 93.0 -> 92.3 mm
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Other:
- board text added: "ESC2"
- board text added: "ESC3"
- board text added: "ESC4"
