File: pcb/FC_v02/FC_v02.kicad_sch (KiCad schematic)
At the start: 86 parts, among them J1 USB_C_Receptacle_USB2.0_16P, J10 2.54mm, J11 2.54mm, J12 JST1.25, J13 JST1.25, J14 Micro_SD_Card_Det1, J2 JST1.25, J3 JST1.25, J4 JST1.25, J5 JST1.25, J6 JST1.25, J8 JST1.25, J9 2.54mm, Q1 SS8050, Q2 SS8050, Q3 Si2301, SW1 BOOT, SW2 USER, SW3 RST, U1 USBLC6-2SC6, U2 CP2102, U3 GY-87, U4 DW01A, U5 8205, U6 AP2112K-3.3, U7 ME6211C33M5, U8 Ai-Thinker-Ra-02, U9 esp32s3_wroom1

Commit message: feat(mag-calib): implement full 3D rotated ellipsoid SIMD calibration and system-wide updates
- Implement 3D rotated and offset ellipsoid fitting (ellipsoid_fit.h/cpp) with Adam optimizer and analytical gradients
- Enforce full hardware SIMD acceleration via Matrix and Vec3 overloaded operators
- Normalize calibrated and filtered magnetometer output to unit sphere for EKF attitude estimation
- Add continuous tumble acquisition with spatial-thinning distance gating in task_calib_mag
- Forward user button clicks from FSM to signal calibration completion
- Add Option 11 to universal_flight_analyzer.py with RMSE convergence and 3D projection plots
- Consolidate firmware Layer 4 core directories (sensor, math, blackbox, telemetry, interface)
- Update Flash NVS storage driver and boot logging for 9-parameter magnetometer calibration
Parts:
- J12, J6: value JST1.25 -> MX1.25; footprint Local Footprints:JST_1.25mm_RA_SMD_4P -> Local Footprints:MX_1.25mm_RA_SMD_4P
- J13: footprint Local Footprints:JST_1.25mm_RA_SMD_2P -> Local Footprints:MX_1.25mm_RA_SMD_2P
- J2, J3, J4, J5: value JST1.25 -> MX1.25; footprint Local Footprints:JST_1.25mm_RA_SMD_3P -> Local Footprints:MX_1.25mm_RA_SMD_3P
- J8: value JST1.25 -> MX1.25; footprint Local Footprints:JST_1.25mm_RA_SMD_8P -> Local Footprints:MX_1.25mm_RA_SMD_8P
- U9: value esp32s3_wroom1 -> esp32-s3-wroom-1-n8-r8
Connections:
- net DRDY: now also U9.35 (IO42); no longer U9.14 (IO20)
- net ESC_PWM1: now also J5.3 (Pin_3), U9.4 (IO4); no longer J4.3 (Pin_3), U9.15 (IO3)
- net ESC_PWM2: now also U9.15 (IO3); no longer U9.13 (IO19)
- net ESC_PWM3: now also J4.3 (Pin_3), U9.33 (IO40); no longer J2.3 (Pin_3), U9.39 (IO1)
- net ESC_PWM4: now also J2.3 (Pin_3), U9.39 (IO1); no longer J5.3 (Pin_3), U9.4 (IO4)
- net RF_RST: now also U9.34 (IO41); no longer U9.35 (IO42)
- net VBEC: now also J3.2 (Pin_2); no longer J4.2 (Pin_2)
- net SCL1 renamed JTAG_D+
- net JTAG_D+: now also U9.14 (IO20); no longer U9.34 (IO41)
- net SDA1 renamed JTAG_D-
- net JTAG_D-: now also U9.13 (IO19); no longer U9.33 (IO40)
Other:
- note added: "I2C1 JTAG"
- note removed: "I2C"
- moved on the sheet: C15, C16, C17, J3, J4, R17
